Commit message: Arreglados problemas de transformaciones con control inexistente de posicion/velocidad, arreglado los paths relativos de los archivos .stl asi se ve bien el robot en la simulacion

File: deepracer_description/models/xacro/control/deepracer_ros_control.xacro (robot description, xacro)
@@ -39,16 +39,20 @@
     <joint name="left_rear_wheel_joint">
       <command_interface name="velocity"/>
+      <state_interface name="position"/>
       <state_interface name="velocity"/>
     </joint>
     <joint name="right_rear_wheel_joint">
       <command_interface name="velocity"/>
+      <state_interface name="position"/>
       <state_interface name="velocity"/>
     </joint>
     <joint name="left_front_wheel_joint">
       <command_interface name="velocity"/>
+      <state_interface name="position"/>
       <state_interface name="velocity"/>
     </joint>
     <joint name="right_front_wheel_joint">
       <command_interface name="velocity"/>
+      <state_interface name="position"/>
       <state_interface name="velocity"/>
     </joint>
@@ -57,4 +61,5 @@
       </command_interface>
       <state_interface name="position"/>
+      <state_interface name="velocity" />
     </joint>
     <joint name="right_steering_hinge_joint">
@@ -62,5 +67,34 @@
       </command_interface>
       <state_interface name="position"/>
+      <state_interface name="velocity" />
     </joint>
+    <!--
+    <joint name="left_rear_wheel_joint">
+      <command_interface name="position"/>
+      <state_interface name="position"/>
+    </joint>
+    <joint name="right_rear_wheel_joint">
+      <command_interface name="position"/>
+      <state_interface name="position"/>
+    </joint>
+    <joint name="left_front_wheel_joint">
+      <command_interface name="position"/>
+      <state_interface name="position"/>
+    </joint>
+    <joint name="right_front_wheel_joint">
+      <command_interface name="position"/>
+      <state_interface name="position"/>
+    </joint>
+    <joint name="left_steering_hinge_joint">
+      <command_interface name="velocity">
+      </command_interface>
+      <state_interface name="velocity"/>
+    </joint>
+    <joint name="right_steering_hinge_joint">
+      <command_interface name="velocity">
+      </command_interface>
+      <state_interface name="velocity"/>
+    </joint>
+    -->
   </ros2_control>
   <gazebo>

File: deepracer_description/models/xacro/deepracer/deepracer.xacro (robot description, xacro)
@@ -25,6 +25,10 @@
   <xacro:arg name="lidar_360_degree_sample" default="600" />
   <xacro:arg name="lidar_360_degree_horizontal_resolution" default="1" />
+  <!--
   <xacro:arg name="lidar_360_degree_min_angle" default="-2.61799" />
   <xacro:arg name="lidar_360_degree_max_angle" default="2.61799" />
+  -->
+  <xacro:arg name="lidar_360_degree_min_angle" default="-3.141592" />
+  <xacro:arg name="lidar_360_degree_max_angle" default="3.141592" />
   <xacro:arg name="lidar_360_degree_min_range" default="0.15" />
   <xacro:arg name="lidar_360_degree_max_range" default="10.0" />

File: deepracer_description/models/xacro/urdf/deepracer_front_facing_camera_and_lidar_urdf.xacro (robot description, xacro)
@@ -23,7 +23,11 @@
         rpy="0 0 0" />
       <mass value="1.9068" />
-	    <inertia ixx="0.004151895" ixy="0"             ixz="0"
-	                               iyy="0.010379737"   iyz="0"
-	                                                   izz="0.010379737" />
+      <inertia
+        ixx="0.004151895"
+        ixy="0"
+        ixz="0"
+        iyy="0.010379737"
+        iyz="0"
+        izz="0.010379737" />
     </inertial>
   </link>
@@ -40,7 +44,11 @@
         rpy="0 1.5707 1.5707" />
      <mass value="0.042222" />
-	   <inertia ixx="0.0000611771" ixy="0"            ixz="0"
-	                               iyy="0.0000611771" iyz="0"
-	                                                  izz="0.0000944606" />
+     <inertia
+        ixx="0.0000611771"
+        ixy="0"
+        ixz="0"
+        iyy="0.0000611771"
+        iyz="0"
+        izz="0.0000944606" />
     </inertial>
     <visual>
@@ -86,7 +94,7 @@
         rpy="0 1.5707 1.5707" />
      <mass value="0.042222" />
-	   <inertia ixx="0.0000611771" ixy="0"            ixz="0"
-	                               iyy="0.0000611771" iyz="0"
-	                                                  izz="0.0000944606" />
+           <inertia ixx="0.0000611771" ixy="0"            ixz="0"
+                                       iyy="0.0000611771" iyz="0"
+                                                          izz="0.0000944606" />
     </inertial>
     <visual>
@@ -146,5 +154,5 @@
       <geometry>
         <mesh
-          filename="package://meshes/left_steering_hinge.STL" />
+          filename="file://$(find deepracer_description)/meshes/left_steering_hinge.STL" />
       </geometry>
     </visual>
@@ -175,7 +183,7 @@
         rpy="0 1.5707 1.5707" />
      <mass value="0.042222" />
-	   <inertia ixx="0.0000611771" ixy="0"            ixz="0"
-	                               iyy="0.0000611771" iyz="0"
-	                                                  izz="0.0000944606" />
+           <inertia ixx="0.0000611771" ixy="0"            ixz="0"
+                                       iyy="0.0000611771" iyz="0"
+                                                          izz="0.0000944606" />
     </inertial>
     <visual>
@@ -235,5 +243,5 @@
       <geometry>
         <mesh
-          filename="package://meshes/right_steering_hinge.STL" />
+          filename="file://$(find deepracer_description)/meshes/right_steering_hinge.STL" />
       </geometry>
     </visual>
@@ -264,7 +272,7 @@
         rpy="0 1.5707 1.5707" />
      <mass value="0.042222" />
-	   <inertia ixx="0.0000611771" ixy="0"            ixz="0"
-	                               iyy="0.0000611771" iyz="0"
-	                                                  izz="0.0000944606" />
+           <inertia ixx="0.0000611771" ixy="0"            ixz="0"
+                                       iyy="0.0000611771" iyz="0"
+                                                          izz="0.0000944606" />
     </inertial>
     <visual>
@@ -326,5 +334,5 @@
         <geometry>
           <mesh
-            filename="package://meshes/zed_camera_link.STL" />
+            filename="file://$(find deepracer_description)/meshes/zed_camera_link.STL" />
         </geometry>
       </visual>
@@ -397,5 +405,5 @@
         <geometry>
           <mesh
-            filename="package://meshes/laser.STL" />
+            filename="file://$(find deepracer_description)/meshes/laser.STL" />
         </geometry>
       </visual>
@@ -407,5 +415,5 @@
       <geometry>
         <mesh
-          filename="package://meshes/laser.STL" />
+          filename="file://$(find deepracer_description)/meshes/laser.STL" />
       </geometry>
     </collision>
@@ -446,5 +454,5 @@
       <geometry>
         <mesh
-          filename="package://meshes/$(arg shell)" />
+          filename="file://$(find deepracer_description)/meshes/$(arg shell)" />
       </geometry>
     </visual>
@@ -455,5 +463,5 @@
       <geometry>
         <mesh
-          filename="package://meshes/$(arg shell)" />
+          filename="file://$(find deepracer_description)/meshes/$(arg shell)" />
       </geometry>
     </collision>
